File: RX_3_ax5043.kicad_sch (KiCad schematic)
At the start: 19 parts, among them P3 CONUFL001-SMD-T, Q5 DMP2160UWQ-7, U17 AX5043

Commit message: Switch the 78nH parts on the RX AX5043 inputs to 75nH
78nH parts are not that available, especially in space ratings, so it
had to change.  I built a simulation and figured out what looks like a
reasonable approximation of the AX5043 (100 ohms differential?) and
changed the 78nH to 75nH and it didn't make a significant difference.

Signed-off-by: Corey Minyard <corey@minyard.net>
Parts:
- L7, L8: value 78nH 2% -> 75nH 2%
Changed lines of the file:
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@@
 			)
 		)
-		(property "Value" "78nH 2%"
+		(property "Value" "75nH 2%"
 			(at 213.868 134.62 90)
 			(effects
@@
 			)
 		)
-		(property "Value" "78nH 2%"
+		(property "Value" "75nH 2%"
 			(at 191.77 120.142 90)
 			(effects
