File: Clocks.kicad_sch (KiCad schematic)
At the start: 13 parts, among them U3 LMK1C1106-Q1, Y2 O 16,0-JT22CT-A-P-3,3-LF

Commit message: Add licensing
Use CERN-OHL-W version 2

Signed-off-by: Corey Minyard <corey@minyard.net>
Other:
- note removed: "CLOCK"
- title: Radiation Tolerant PacSat Communication -> Clock and Distribution
Changed lines of the file:
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@@
 	(paper "USLedger")
 	(title_block
-		(title "Radiation Tolerant PacSat Communication")
-		(date "2023-06-17")
-		(rev "A")
+		(title "Clock and Distribution")
+		(date "2026-08-20")
+		(rev "4.0")
 		(company "AMSAT-NA")
-		(comment 1 "N5BRG")
+		(comment 1 "AE5KM")
+		(comment 2 "Copyright Corey Minyard, 2026")
+		(comment 3 "Licensed under CERN-OHL-W version 2")
 	)
 	(text "This chip does not have a thermal pad on the\nchip, but does have one in the footprint.\nJust apply solder paste normally there so the\nchip will sit on it and have some thermal\npath to the board besides the pins."
@@
 		)
 	)
-	(text "CLOCK"
-		(exclude_from_sim no)
-		(at 336.55 246.38 0)
-		(effects
-			(font
-				(size 1.524 1.524)
-			)
-			(justify left bottom)
-		)
-	)
