File: Clocks.kicad_sch (KiCad schematic)
At the start: 13 parts, among them U3 LMK1C1106-Q1, Y2 O 16,0-JT22CT-A-P-3,3-LF

Commit message: Change all instances of K (for kilo) to k
That's the standard.

Signed-off-by: Corey Minyard <corey@minyard.net>
Parts:
- FB2, FB3: value 1KΩ@100MHz -> 1kΩ@100MHz
- R121, R25: value 10KΩ -> 10kΩ
- R139: value 10KΩ 1% -> 10kΩ 1%
- TH5: value NTCG103JF103FTDS 10KΩ@25C -> NTCG103JF103FTDS 10kΩ@25C
Other:
- note added: "Thermsistor varies from 534 ohms (125C) to 188.5kΩ (-40C). With a 10kΩ bias this gives a .17 to 3.13V range."
- note removed: "Thermsistor varies from 534 ohms (125C) to 188.5KΩ (-40C). With a 10KΩ bias this gives a .17 to 3.13V range."
Changed lines of the file:
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@@
 		)
 	)
-	(text "Thermsistor varies from 534\nohms (125C) to 188.5KΩ (-40C).\nWith a 10KΩ bias this gives a\n.17 to 3.13V range."
+	(text "Thermsistor varies from 534\nohms (125C) to 188.5kΩ (-40C).\nWith a 10kΩ bias this gives a\n.17 to 3.13V range."
 		(exclude_from_sim no)
 		(at 131.572 160.528 0)
@@
 			)
 		)
-		(property "Value" "1KΩ@100MHz"
+		(property "Value" "1kΩ@100MHz"
 			(at 158.75 90.1318 0)
 			(show_name no)
@@
 			)
 		)
-		(property "Value" "10KΩ 1%"
+		(property "Value" "10kΩ 1%"
 			(at 139.954 168.402 0)
 			(show_name no)
@@
 			)
 		)
-		(property "Value" "10KΩ"
+		(property "Value" "10kΩ"
 			(at 195.072 100.203 0)
 			(show_name no)
@@
 			)
 		)
-		(property "Value" "10KΩ"
+		(property "Value" "10kΩ"
 			(at 141.478 101.473 0)
 			(show_name no)
@@
 			)
 		)
-		(property "Value" "1KΩ@100MHz"
+		(property "Value" "1kΩ@100MHz"
 			(at 215.9 83.1469 0)
 			(show_name no)
@@
 			)
 		)
-		(property "Value" "NTCG103JF103FTDS 10KΩ@25C"
+		(property "Value" "NTCG103JF103FTDS 10kΩ@25C"
 			(at 157.226 188.214 90)
 			(show_name no)

Commit message: Switch out the oscillator with a higher precision one
Signed-off-by: Corey Minyard <corey@minyard.net>
Parts:
- Y2: value O 16,0-JT22CT-A-P-3,3-LF -> TG2520SMN 16.0000M-MCGNNM3
Other:
- note added: "Idd = 1.5mA"
- note removed: "Idd = 5.0 mA"
Changed lines of the file:
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@@
 		)
 	)
-	(text "Idd = 5.0 mA"
+	(text "Idd = 1.5mA"
 		(exclude_from_sim no)
 		(at 160.02 119.38 0)
@@
 		(dnp no)
 		(property "Reference" "Y2"
-			(at 166.37 100.33 0)
-			(show_name no)
-			(do_not_autoplace no)
-			(effects
-				(font
-					(size 1.27 1.27)
-				)
-			)
-		)
-		(property "Value" "O 16,0-JT22CT-A-P-3,3-LF"
-			(at 176.276 103.124 0)
-			(show_name no)
-			(do_not_autoplace no)
+			(at 163.322 102.87 0)
+			(show_name no)
+			(do_not_autoplace no)
+			(effects
+				(font
+					(size 1.27 1.27)
+				)
+			)
+		)
+		(property "Value" "TG2520SMN 16.0000M-MCGNNM3"
+			(at 172.466 100.33 0)
+			(show_name no)
+			(do_not_autoplace no)

Commit message: DNP the oscillator control resistor
The new oscillator requires the VC pin to float.  But leave it in
in case the oscillator needs to change.

Signed-off-by: Corey Minyard <corey@minyard.net>
Parts:
- R25: now not fitted; now left out of the parts list
Other:
- note added: "Some oscillators use the VC input as an enable, some use it as a voltage control, and some don't use it and require it to float. The current requires it to float, but leave R25 here in case the oscillator needs to change."
Changed lines of the file:
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@@
+		)
+	)
+	(text "Some oscillators use the VC input as an enable,\nsome use it as a voltage control, and some don't\nuse it and require it to float.  The current\nrequires it to float, but leave R25 here in\ncase the oscillator needs to change."
+		(exclude_from_sim no)
+		(at 101.854 86.614 0)
+		(effects
+			(font
+				(size 1.524 1.524)
+			)
 		)
 	)
@@
 		(body_style 1)
 		(exclude_from_sim no)
-		(in_bom yes)
+		(in_bom no)
 		(on_board yes)
 		(in_pos_files yes)
-		(dnp no)
+		(dnp yes)
 		(property "Reference" "R25"
 			(at 141.478 99.1616 0)
