File: PacSat_AFSK.kicad_sch (KiCad schematic)
At the start: 18 parts

Commit message: Add licensing
Use CERN-OHL-W version 2

Signed-off-by: Corey Minyard <corey@minyard.net>
Other:
- title: Radiation Tolerant Internal Housekeeping Unit (IHU) -> PacSat Radio and Control Board
Changed lines of the file:
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@@
 	(paper "USLedger")
 	(title_block
-		(title "Radiation Tolerant Internal Housekeeping Unit (IHU)")
-		(date "2022-12-27")
-		(rev "1.2")
+		(title "PacSat Radio and Control Board")
+		(date "2026-08-20")
+		(rev "4.0")
 		(company "AMSAT-NA")
-		(comment 1 "N5BRG")
+		(comment 1 "AE5KM")
+		(comment 2 "Copyright Corey Minyard, 2026")
+		(comment 3 "Licensed under CERN-OHL-W version 2")
 	)
 	(text "These holes are for if you solder a cable\nonto the antenna connector pad.  The are\nfor a 2.4mm Tefzel ETFE zip tie to provide\nstrain relief for the cable."
