File: ax5043.kicad_sch (KiCad schematic)
At the start: 0 parts

Commit message: Add licensing
Use CERN-OHL-W version 2

Signed-off-by: Corey Minyard <corey@minyard.net>
Other:
- company: (none) -> AMSAT-NA
- title: (none) -> All AX5043 Radios
Changed lines of the file:
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@@
 	(generator_version "10.0")
 	(paper "A4")
+	(title_block
+		(title "All AX5043 Radios")
+		(date "2026-08-20")
+		(rev "4.0")
+		(company "AMSAT-NA")
+		(comment 1 "AE5KM")
+		(comment 2 "Copyright Corey Minyard, 2026")
+		(comment 3 "Licensed under CERN-OHL-W version 2")
+	)
 	(sheet
 		(at 105.41 31.75)
