File: rf_in_switch.kicad_sch (KiCad schematic)
At the start: 6 parts, among them P17 MMCX-J-P-H-RA-TH1, P18 CONUFL001-SMD-T, U31 QPC8010QTR7

Commit message: Add licensing
Use CERN-OHL-W version 2

Signed-off-by: Corey Minyard <corey@minyard.net>
Other:
- company: (none) -> AMSAT-NA
- title: (none) -> RF Input Swtich Controlled by Active Standby
Changed lines of the file:
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@@
 	(generator_version "10.0")
 	(paper "A4")
+	(title_block
+		(title "RF Input Swtich Controlled by Active Standby")
+		(date "2026-08-20")
+		(rev "4.0")
+		(company "AMSAT-NA")
+		(comment 1 "AE5KM")
+		(comment 2 "Copyright Corey Minyard, 2026")
+		(comment 3 "Licensed under CERN-OHL-W version 2")
+	)
 	(text "RX FROM BOARD2"
 		(exclude_from_sim no)

Commit message: Add design notes for outgassing, change board 1-2 connectors to MMCX
Signed-off-by: Corey Minyard <corey@minyard.net>
Parts:
- removed P18: CONUFL001-SMD-T, PacSatDev_misc:CONN1_CONUFL_TEC, symbol PACSAT_DEV_misc:U_FL
- added P26: MMCX-J-P-H-RA-TH1, PacSatDev_misc:COAX4_MMCX-J-P-H-RA-TH1_SAI, symbol PACSAT_DEV_misc:MMCX-J-P-H-RA-TH1
Connections:
- net GND: now also P26.2 (GND), P26.3 (GND), P26.4 (GND), P26.5 (GND)
- net at U31.11 (RF2): now also P26.1 (SIGNAL)
