File: rf_in_switch.kicad_sch (KiCad schematic)
At the start: 6 parts, among them P17 MMCX-J-P-H-RA-TH1, P26 MMCX-J-P-H-RA-TH1, U31 QPC8010QTR7

Commit message: Change all instances of K (for kilo) to k
That's the standard.

Signed-off-by: Corey Minyard <corey@minyard.net>
Parts:
- R97: value 10KΩ -> 10kΩ
Changed lines of the file:
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@@
 			)
 		)
-		(property "Value" "10KΩ"
+		(property "Value" "10kΩ"
 			(at 145.923 163.576 90)
 			(show_name no)
