File: active_standby.kicad_sch (KiCad schematic)
At the start: 21 parts, among them Q10 2N7002TQ-7-F, Q11 2N7002TQ-7-F, Q2 2N7002TQ-7-F, Q8 2N7002TQ-7-F, U24 SN3257QDYYRQ1, U30 SN3257QDYYRQ1

Commit message: Change all instances of K (for kilo) to k
That's the standard.

Signed-off-by: Corey Minyard <corey@minyard.net>
Parts:
- R101, R191, R93: value 18KΩ -> 18kΩ
- R103, R108, R132, R133, R185, R91, R92, R94, R95: value 10KΩ -> 10kΩ
Changed lines of the file:
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@@
 			)
 		)
-		(property "Value" "10KΩ"
+		(property "Value" "10kΩ"
 			(at 38.608 95.123 0)
 			(show_name no)
@@
 			)
 		)
-		(property "Value" "10KΩ"
+		(property "Value" "10kΩ"
 			(at 151.638 27.813 0)
 			(show_name no)
@@
 			)
 		)
-		(property "Value" "10KΩ"
+		(property "Value" "10kΩ"
 			(at 167.132 143.383 0)
 			(show_name no)
@@
 			)
 		)
-		(property "Value" "10KΩ"
+		(property "Value" "10kΩ"
 			(at 236.728 120.523 0)
 			(show_name no)
@@
 			)
 		)
-		(property "Value" "10KΩ"
+		(property "Value" "10kΩ"
 			(at 131.318 97.663 0)
 			(show_name no)
@@
 			)
 		)
-		(property "Value" "10KΩ"
+		(property "Value" "10kΩ"
 			(at 236.728 105.283 0)
 			(show_name no)
@@
 			)
 		)
-		(property "Value" "10KΩ"
+		(property "Value" "10kΩ"
 			(at 142.748 177.673 0)
 			(show_name no)
@@
 			)
 		)
-		(property "Value" "18KΩ"
+		(property "Value" "18kΩ"
 			(at 131.318 117.983 0)
 			(show_name no)
@@
 			)
 		)
-		(property "Value" "18KΩ"
+		(property "Value" "18kΩ"
 			(at 38.608 110.363 0)
 			(show_name no)
@@
 			)
 		)
-		(property "Value" "10KΩ"
+		(property "Value" "10kΩ"
 			(at 175.768 55.753 0)
 			(show_name no)
@@
 			)
 		)
-		(property "Value" "18KΩ"
+		(property "Value" "18kΩ"
 			(at 151.638 39.243 0)
 			(show_name no)
@@
 			)
 		)
-		(property "Value" "10KΩ"
+		(property "Value" "10kΩ"
 			(at 165.608 111.633 0)
 			(show_name no)
