File: diplexer.kicad_sch (KiCad schematic)
At the start: 9 parts, among them P25 MMCX-J-P-H-RA-TH1

Commit message: Add licensing
Use CERN-OHL-W version 2

Signed-off-by: Corey Minyard <corey@minyard.net>
Other:
- company: (none) -> AMSAT-NA
- title: (none) -> Diplexer for Sharing an Antenna
Changed lines of the file:
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@@
 	(generator_version "10.0")
 	(paper "A4")
+	(title_block
+		(title "Diplexer for Sharing an Antenna")
+		(date "2026-08-20")
+		(rev "4.0")
+		(company "AMSAT-NA")
+		(comment 1 "AE5KM")
+		(comment 2 "Copyright Corey Minyard, 2026")
+		(comment 3 "Licensed under CERN-OHL-W version 2")
+	)
 	(text "Inductor to bleed off static build\nup on the antenna."
 		(exclude_from_sim no)

Commit message: Change all instances of K (for kilo) to k
That's the standard.

Signed-off-by: Corey Minyard <corey@minyard.net>
Parts:
- R123: value 10KΩ -> 10kΩ
Changed lines of the file:
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@@
 			)
 		)
-		(property "Value" "10KΩ"
+		(property "Value" "10kΩ"
 			(at 125.603 125.476 90)
 			(show_name no)
